File: output/pcbs/main.kicad_pcb (KiCad board)
At the start: 2 copper layers, 444 x 183.4 mm, 136 parts

Commit message: Route diodes, switches
Routing:
- net MRST: track 0.00 -> 61.9 mm, vias 0 -> 1
- net GND: track 0.00 -> 44.1 mm
- net MGND: track 0.00 -> 37.3 mm
- net MRAW: track 0.00 -> 34.2 mm
- net PP7: track 0.00 -> 27.3 mm
- net P14: track 0.00 -> 27.3 mm
- net MP16: track 0.00 -> 26.3 mm
- net MP9: track 0.00 -> 25.9 mm
- net MP8: track 0.00 -> 25.9 mm
- net MP10: track 0.00 -> 25.9 mm
- net P9: track 0.00 -> 25.9 mm
- net P8: track 0.00 -> 25.9 mm
- net P16: track 0.00 -> 25.9 mm
- net P10: track 0.00 -> 25.9 mm
- net RST: track 0.00 -> 21.4 mm
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Other:
- net class Default removed
