File: output/pcbs/main.kicad_pcb (KiCad board)
At the start: 2 copper layers, 444 x 183.4 mm, 136 parts

Commit message: Finish wiring
Connections:
- D55 pad 1: PP7 -> MP7
- D56 pad 1: PP7 -> MP7
- D57 pad 1: PP7 -> MP7
- D58 pad 1: PP7 -> MP7
- D59 pad 1: PP7 -> MP7
- D60 pad 1: PP7 -> MP7
- S5 pad 1: P23 -> P3
- S6 pad 1: P23 -> P3
- S7 pad 1: P23 -> P3
- S8 pad 1: P23 -> P3
Routing:
- net P2: track 0.00 -> 283.2 mm, vias 0 -> 3
- net P3: track 0.00 -> 276.3 mm, vias 0 -> 3
- net MP21: track 0.00 -> 273.3 mm, vias 0 -> 3
- net P4: track 0.00 -> 273.0 mm, vias 0 -> 3
- net MP20: track 0.00 -> 267.9 mm, vias 0 -> 3
- net P5: track 0.00 -> 265.2 mm, vias 0 -> 3
- net MP19: track 0.00 -> 257.5 mm, vias 0 -> 3
- net P6: track 0.00 -> 256.6 mm, vias 0 -> 3
- net MP18: track 0.00 -> 248.8 mm, vias 0 -> 3
- net P7: track 0.00 -> 247.6 mm, vias 0 -> 3
- net MP15: track 0.00 -> 240.0 mm, vias 0 -> 3
- net MP14: track 0.00 -> 232.3 mm, vias 0 -> 3
- net MP7: track 0.00 -> 219.3 mm, vias 0 -> 2
- net P14: track 27.3 -> 212.0 mm, vias 0 -> 2
- net P16: track 25.9 -> 183.1 mm
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- added copper zone on B.Cu, net GND
- added copper zone on F.Cu, net GND
- added copper zone on B.Cu, net MGND
- added copper zone on F.Cu, net MGND

Commit message: Change template for pcb
Parts:
- moved D31 144.0 mm to (376.0, 105.0)
- moved D32 144.0 mm to (376.0, 88.0)
- moved D33 144.0 mm to (376.0, 71.0)
- moved D34 144.0 mm to (376.0, 54.0)
- moved D35 144.0 mm to (358.0, 105.0)
- moved D36 144.0 mm to (358.0, 88.0)
- moved D37 144.0 mm to (358.0, 71.0)
- moved D38 144.0 mm to (358.0, 54.0)
- moved D39 144.0 mm to (340.0, 100.0)
- moved D40 144.0 mm to (340.0, 83.0)
- moved D41 144.0 mm to (340.0, 66.0)
- moved D42 144.0 mm to (340.0, 49.0)
- moved D43 144.0 mm to (322.0, 97.5)
- moved D44 144.0 mm to (322.0, 80.5)
- moved D45 144.0 mm to (322.0, 63.5)
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Connections:
- D55 pad 1: MP7 -> PP7
- D56 pad 1: MP7 -> PP7
- D57 pad 1: MP7 -> PP7
- D58 pad 1: MP7 -> PP7
- D59 pad 1: MP7 -> PP7
- D60 pad 1: MP7 -> PP7
- S5 pad 1: P3 -> P23
- S6 pad 1: P3 -> P23
- S7 pad 1: P3 -> P23
- S8 pad 1: P3 -> P23
Routing:
- net P2: track 283.2 -> 0.00 mm, vias 3 -> 0
- net P3: track 276.3 -> 0.00 mm, vias 3 -> 0
- net MP21: track 273.3 -> 0.00 mm, vias 3 -> 0
- net P4: track 273.0 -> 0.00 mm, vias 3 -> 0
- net MP20: track 267.9 -> 0.00 mm, vias 3 -> 0
- net P5: track 265.2 -> 0.00 mm, vias 3 -> 0
- net MP19: track 257.5 -> 0.00 mm, vias 3 -> 0
- net P6: track 256.6 -> 0.00 mm, vias 3 -> 0
- net MP18: track 248.8 -> 0.00 mm, vias 3 -> 0
- net P7: track 247.6 -> 0.00 mm, vias 3 -> 0
- net MP15: track 240.0 -> 0.00 mm, vias 3 -> 0
- net MP14: track 232.3 -> 0.00 mm, vias 3 -> 0
- net MP7: track 219.3 -> 0.00 mm, vias 2 -> 0
- net P14: track 212.0 -> 27.3 mm, vias 2 -> 0
- net P16: track 183.1 -> 25.9 mm
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- removed copper zone on B.Cu, net GND
- removed copper zone on F.Cu, net GND
- removed copper zone on B.Cu, net MGND
- removed copper zone on F.Cu, net MGND
Other:
- board size 444 x 183.4 mm -> 300 x 183.4 mm

Commit message: Fix net names
Connections:
- D55 pad 1: PP7 -> MP7
- D56 pad 1: PP7 -> MP7
- D57 pad 1: PP7 -> MP7
- D58 pad 1: PP7 -> MP7
- D59 pad 1: PP7 -> MP7
- D60 pad 1: PP7 -> MP7
- S5 pad 1: P23 -> P3
- S6 pad 1: P23 -> P3
- S7 pad 1: P23 -> P3
- S8 pad 1: P23 -> P3
Routing:
- net MRST: track 52.8 -> 0.00 mm, vias 1 -> 0
- net GND: track 43.1 -> 0.00 mm
- net MGND: track 37.3 -> 0.00 mm
- net MRAW: track 32.3 -> 0.00 mm
- net PP7: track 27.3 -> 0.00 mm
- net P14: track 27.3 -> 0.00 mm
- net MP9: track 25.9 -> 0.00 mm
- net MP8: track 25.9 -> 0.00 mm
- net MP16: track 25.9 -> 0.00 mm
- net MP10: track 25.9 -> 0.00 mm
- net P9: track 25.9 -> 0.00 mm
- net P8: track 25.9 -> 0.00 mm
- net P16: track 25.9 -> 0.00 mm
- net P10: track 25.9 -> 0.00 mm
- net RST: track 21.0 -> 0.00 mm
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
Commit message: Start (hopefully final) pass
Routing:
- net MP9: track 0.00 -> 25.9 mm
- net MP8: track 0.00 -> 25.9 mm
- net MP16: track 0.00 -> 25.9 mm
- net MP10: track 0.00 -> 25.9 mm
- net P9: track 0.00 -> 25.9 mm
- net P8: track 0.00 -> 25.9 mm
- net P16: track 0.00 -> 25.9 mm
- net P10: track 0.00 -> 25.9 mm
- net mirror_middle_top: track 0.00 -> 4.32 mm
- net mirror_middle_num: track 0.00 -> 4.32 mm
- net mirror_middle_home: track 0.00 -> 4.32 mm
- net mirror_middle_bottom: track 0.00 -> 4.32 mm
- net middle_num: track 0.00 -> 4.32 mm
- net inner_top: track 0.00 -> 4.32 mm
- net inner_home: track 0.00 -> 4.32 mm
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
Commit message: Finish switch-local wiring
Routing:
- net MP7: track 0.00 -> 27.3 mm
- net P14: track 0.00 -> 27.3 mm
- net mirror_fourth_cluster: track 0.00 -> 16.1 mm
- net mirror_sixth_cluster: track 0.00 -> 16.0 mm
- net sixth_cluster: track 0.00 -> 16.0 mm
- net mirror_second_cluster: track 0.00 -> 15.4 mm
- net fourth_cluster: track 0.00 -> 15.4 mm
- net second_cluster: track 0.00 -> 15.3 mm
- net first_cluster: track 0.00 -> 15.3 mm
- net third_cluster: track 0.00 -> 15.3 mm
- net mirror_first_cluster: track 0.00 -> 15.1 mm
- net mirror_third_cluster: track 0.00 -> 15.1 mm
- net mirror_fifth_cluster: track 0.00 -> 14.9 mm
- net fifth_cluster: track 0.00 -> 14.9 mm
- net mirror_ring_top: track 4.32 -> 14.9 mm
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
Commit message: Matrix column wiring
Routing:
- net P7: track 0.00 -> 78.7 mm
- net P6: track 0.00 -> 78.3 mm
- net P5: track 0.00 -> 78.3 mm
- net P4: track 0.00 -> 77.6 mm
- net P2: track 0.00 -> 77.6 mm
- net P3: track 0.00 -> 77.6 mm
- net MP19: track 0.00 -> 74.0 mm
- net MP21: track 0.00 -> 73.7 mm
- net MP18: track 0.00 -> 73.7 mm
- net MP14: track 0.00 -> 73.7 mm
- net MP15: track 0.00 -> 73.7 mm
- net MP20: track 0.00 -> 73.5 mm

Commit message: Fix DRC, add copper fills + vias to connect isolated fills
Routing:
- net P4: track 77.6 -> 306.0 mm, vias 0 -> 2
- net MP7: track 27.3 -> 242.3 mm
- net MP19: track 74.0 -> 282.6 mm, vias 0 -> 2
- net P2: track 77.6 -> 284.3 mm
- net P14: track 27.3 -> 226.6 mm
- net P5: track 78.3 -> 277.5 mm, vias 0 -> 2
- net P3: track 77.6 -> 275.1 mm
- net MP21: track 73.7 -> 267.2 mm
- net P6: track 78.3 -> 263.4 mm, vias 0 -> 2
- net MP18: track 73.7 -> 257.4 mm, vias 0 -> 2
- net MP20: track 73.5 -> 253.9 mm
- net P7: track 78.7 -> 253.0 mm, vias 0 -> 2
- net MP15: track 73.7 -> 246.4 mm, vias 0 -> 2
- net MP14: track 73.7 -> 234.4 mm, vias 0 -> 2
- net P16: track 25.9 -> 179.6 mm
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- added copper zone on B.Cu, net GND
- added copper zone on F.Cu, net GND
- added copper zone on B.Cu, net MGND
- added copper zone on F.Cu, net MGND

Commit message: Fill out case code, get converted stls
Routing:
- net P4: track 306.0 -> 0.00 mm, vias 2 -> 0
- net P2: track 284.3 -> 0.00 mm
- net MP19: track 282.6 -> 0.00 mm, vias 2 -> 0
- net P5: track 277.5 -> 0.00 mm, vias 2 -> 0
- net P3: track 275.1 -> 0.00 mm
- net MP21: track 267.2 -> 0.00 mm
- net P6: track 263.4 -> 0.00 mm, vias 2 -> 0
- net MP18: track 257.4 -> 0.00 mm, vias 2 -> 0
- net MP20: track 253.9 -> 0.00 mm
- net P7: track 253.0 -> 0.00 mm, vias 2 -> 0
- net MP15: track 246.4 -> 0.00 mm, vias 2 -> 0
- net MP7: track 242.3 -> 0.00 mm
- net MP14: track 234.4 -> 0.00 mm, vias 2 -> 0
- net P14: track 226.6 -> 0.00 mm
- net P16: track 179.6 -> 0.00 mm
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- removed copper zone on B.Cu, net GND
- removed copper zone on F.Cu, net GND
- removed copper zone on B.Cu, net MGND
- removed copper zone on F.Cu, net MGND
